File: physical2/amtdoor2v2.sch (KiCad schematic (older format))
At the start: 77 parts, among them J1 RJ45, J2 RJ45, P1 CONN_02X23, P2 CONN_02X23, P3 CONN_01X02, P4 CONN_01X02, P5 CONN_01X05, Q1 Q_NPN_BCE, Q2 Q_NMOS_DGS, T1 H2019FNL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

Commit message: Fix PoE schematic, make major footprints, begin board grouping.
* Swap RJ45 output for 2x3 .1" header. Use either small pcb or custom cable to connect to BBB.
* Add footprints for ethernet jacks, transformers, large diodes/inductors, optoisolators, solder bridge.
* Fix direction of optoisolator in feedback.
* Fix power nFET symbol.
* Fix incorrect ground on RJ45 shields.
* Build symbol <-> footprint cmp file.

Todo:
* Check capacitor/resistor sizes. Set to 0805 by default.
* Check diode direction and pin mappings. Fishy.
Parts:
- removed J2: RJ45, symbol RJ45
- removed Q2: Q_NMOS_DGS, symbol Q_NMOS_DGS
- removed U2, U3, U4: TLP785F, DIP-4F, symbol TLP785F
- added P6: CONN_02X03, symbol CONN_02X03
- added Q2: FDC2612, symbol FDC2612
- added U2, U3: MOCD217M, symbol OPTO-TRANSISTOR-2
- C1: value 0.1uF -> 0.1uF 100V 1206
- D3: value D_Schottky_Small -> Schottky 58V SMA
- gave numbers to parts that had none: 9
Connections:
- wire segments 345 -> 277
Other:
- note added: "Stackable Female: Samtec Inc SSQ-123-03-T-D"
- note removed: "Samtec Inc SSQ-123-03-T-D"
